File: ESP32_S2_SOLO_N4 Kicad Reference Design.kicad_pcb (KiCad board)
At the start: 2 copper layers, 0 parts

Commit message: Layout done
Parts:
- added C1: 100nF, Capacitor_SMD:C_0805_2012Metric_Pad1.18x1.45mm_HandSolder, F.Cu at (127.0, 43.5)
- added C2: 10uF, Capacitor_SMD:C_0805_2012Metric_Pad1.18x1.45mm_HandSolder, F.Cu at (134.0, 43.5)
- added C3: .1uF, Capacitor_SMD:C_0805_2012Metric_Pad1.18x1.45mm_HandSolder, F.Cu at (141.5, 43.5)
- added C4: .1uF, Capacitor_SMD:C_0805_2012Metric_Pad1.18x1.45mm_HandSolder, F.Cu at (148.5, 43.5)
- added C5: 1uF, Capacitor_SMD:C_0805_2012Metric_Pad1.18x1.45mm_HandSolder, F.Cu at (156.0, 43.5)
- added C6: .1uF, Capacitor_SMD:C_0805_2012Metric_Pad1.18x1.45mm_HandSolder, F.Cu at (163.0, 43.5)
- added D1: 1N4148WT, Diode_SMD:D_0805_2012Metric_Pad1.15x1.40mm_HandSolder, F.Cu at (145.0, 146.5)
- added J2: USB_C_Receptacle_USB2.0, Connector_USB:USB_C_Receptacle_GCT_USB4105-xx-A_16P_TopMnt_Horizontal, F.Cu at (100.3, 65.4)
- added LD1: SPL_PL90, Connector_PinSocket_2.54mm:PinSocket_1x02_P2.54mm_Vertical, F.Cu at (162.5, 128.0)
- added LD2: SPL_PL90, Connector_PinSocket_2.54mm:PinSocket_1x02_P2.54mm_Vertical, F.Cu at (162.5, 120.5)
- added LD3: SPL_PL90, Connector_PinSocket_2.54mm:PinSocket_1x02_P2.54mm_Vertical, F.Cu at (162.5, 113.0)
- added LD4: SPL_PL90, Connector_PinSocket_2.54mm:PinSocket_1x02_P2.54mm_Vertical, F.Cu at (162.5, 105.5)
- added LD5: SPL_PL90, Connector_PinSocket_2.54mm:PinSocket_1x02_P2.54mm_Vertical, F.Cu at (162.5, 98.0)
- added LD6: SPL_PL90, Connector_PinSocket_2.54mm:PinSocket_1x02_P2.54mm_Vertical, F.Cu at (162.5, 90.5)
- added LD7: SPL_PL90, Connector_PinSocket_2.54mm:PinSocket_1x02_P2.54mm_Vertical, F.Cu at (162.5, 83.0)
- added LS1: Speaker, Connector_PinSocket_2.54mm:PinSocket_1x02_P2.54mm_Vertical, F.Cu at (145.0, 136.5)
- added Q1: NPN, Package_TO_SOT_SMD:TSOT-23_HandSoldering, F.Cu at (182.5, 83.0)
- added R1: 10k, Resistor_SMD:R_0805_2012Metric_Pad1.20x1.40mm_HandSolder, F.Cu at (126.0, 64.5)
- added R10: 60k, Resistor_SMD:R_0805_2012Metric_Pad1.20x1.40mm_HandSolder, F.Cu at (116.0, 113.0)
- added R11: 91, Resistor_SMD:R_0805_2012Metric_Pad1.20x1.40mm_HandSolder, F.Cu at (162.5, 69.0)
- added R12: 60k, Resistor_SMD:R_0805_2012Metric_Pad1.20x1.40mm_HandSolder, F.Cu at (107.0, 82.0)
- added R13: 180k, Resistor_SMD:R_0805_2012Metric_Pad1.20x1.40mm_HandSolder, F.Cu at (101.0, 82.5)
- added R14: R_Photo, Connector_PinSocket_2.54mm:PinSocket_1x02_P2.54mm_Vertical, F.Cu at (128.0, 105.5)
- added R15: 60k, Resistor_SMD:R_0805_2012Metric_Pad1.20x1.40mm_HandSolder, F.Cu at (116.0, 105.5)
- added R16: R_Photo, Connector_PinSocket_2.54mm:PinSocket_1x02_P2.54mm_Vertical, F.Cu at (128.0, 98.0)
- added R17: 60k, Resistor_SMD:R_0805_2012Metric_Pad1.20x1.40mm_HandSolder, F.Cu at (116.0, 98.0)
- added R18: R_Photo, Connector_PinSocket_2.54mm:PinSocket_1x02_P2.54mm_Vertical, F.Cu at (128.0, 90.5)
- added R19: 60k, Resistor_SMD:R_0805_2012Metric_Pad1.20x1.40mm_HandSolder, F.Cu at (116.0, 90.5)
- added R2: 5.1 k, Resistor_SMD:R_0805_2012Metric_Pad1.20x1.40mm_HandSolder, F.Cu at (126.0, 58.5)
- added R20: R_Photo, Connector_PinSocket_2.54mm:PinSocket_1x02_P2.54mm_Vertical, F.Cu at (128.0, 82.5)
- added R21: 60k, Resistor_SMD:R_0805_2012Metric_Pad1.20x1.40mm_HandSolder, F.Cu at (116.0, 82.5)
- added R3: 5.1 k, Resistor_SMD:R_0805_2012Metric_Pad1.20x1.40mm_HandSolder, F.Cu at (126.0, 70.0)
- added R4: 60k, Resistor_SMD:R_0805_2012Metric_Pad1.20x1.40mm_HandSolder, F.Cu at (116.0, 128.0)
- added R5: R_Photo, Connector_PinSocket_2.54mm:PinSocket_1x02_P2.54mm_Vertical, F.Cu at (128.0, 128.0)
- added R6: R_Variable, Resistor_THT:R_Axial_DIN0207_L6.3mm_D2.5mm_P15.24mm_Horizontal, F.Cu at (184.5, 58.5)
- added R7: R_Photo, Connector_PinSocket_2.54mm:PinSocket_1x02_P2.54mm_Vertical, F.Cu at (128.0, 120.5)
- added R8: 60k, Resistor_SMD:R_0805_2012Metric, F.Cu at (116.1, 120.5)
- added R9: R_Photo, Connector_PinSocket_2.54mm:PinSocket_1x02_P2.54mm_Vertical, F.Cu at (128.0, 113.0)
- added REF**: MountingHole_3.2mm_M3, MountingHole:MountingHole_3.2mm_M3, F.Cu at (105.0, 141.0)
- added REF**: MountingHole_3.2mm_M3, MountingHole:MountingHole_3.2mm_M3, F.Cu at (183.0, 141.0)
- added REF**: MountingHole_3.2mm_M3, MountingHole:MountingHole_3.2mm_M3, F.Cu at (105.0, 48.0)
- added REF**: MountingHole_3.2mm_M3, MountingHole:MountingHole_3.2mm_M3, F.Cu at (183.0, 48.0)
- added SW1: Reset, footprints 2:SWDIP2_256X170P100, F.Cu at (131.0, 52.5)
- added SW2: Boot, footprints 2:SWDIP2_256X170P100, F.Cu at (166.0, 52.5)
- added SW3: SW_SPDT, Button_Switch_SMD:SW_DPDT_CK_JS202011JCQN, F.Cu at (174.5, 63.3)
- added SW5: SW_SPDT, Button_Switch_SMD:SW_DPDT_CK_JS202011JCQN, F.Cu at (174.5, 68.8)
- added U1: ESP32-S2-SOLO, ESP32_S2_SOLO_N4:XCVR_ESP32-S2-SOLO-N4, F.Cu at (144.6, 63.0)
- added U10: LM339DR, footprints:D14, F.Cu at (153.5, 138.0)
- added U2: LD1117S33TR_SOT223, Package_TO_SOT_SMD:SOT-223-3_TabPin2, F.Cu at (116.0, 65.5)
- added U3: LM339DR, footprints:D14, F.Cu at (136.5, 137.8)
Routing:
- net GND: track 0.00 -> 347.5 mm, vias 0 -> 2
- net +3.3V: track 0.00 -> 219.5 mm, vias 0 -> 2
- net /3.3V_0.75: track 0.00 -> 115.3 mm, vias 0 -> 2
- net /D6: track 0.00 -> 106.5 mm, vias 0 -> 2
- net /A3: track 0.00 -> 104.7 mm, vias 0 -> 2
- net Net-(D1-K): track 0.00 -> 100.8 mm
- net Net-(D1-A): track 0.00 -> 93.4 mm, vias 0 -> 2
- net /A0: track 0.00 -> 84.8 mm
- net /A1: track 0.00 -> 78.1 mm
- net /A2: track 0.00 -> 76.9 mm, vias 0 -> 2
- net /A4: track 0.00 -> 76.3 mm, vias 0 -> 2
- net /A5: track 0.00 -> 75.1 mm
- net /A6: track 0.00 -> 73.9 mm
- net /3.3V_Switch: track 0.00 -> 69.8 mm
- net /D5: track 0.00 -> 69.7 mm, vias 0 -> 2
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- added copper zone on B.Cu, net GND
- added copper zone on F.Cu, net GND
Other:
- board outline added: 95 x 110 mm
