File: ESP32_S2_SOLO_N4 Kicad Reference Design.kicad_sch (KiCad schematic)
At the start: 52 parts, among them J2 USB_C_Receptacle_USB2.0, Q1 NPN, SW1 Reset, SW2 Boot, SW3 SW_Nidec_CAS-120A1, SW4 SW_Nidec_CAS-120A1, U1 ESP32-S2-SOLO, U10 LM339DR, U2 LD1117S33TR_SOT223, U3 LM339DR

Commit message: Footprints done
Parts:
- removed R22, R23, R24, R25, R26, R27: R, symbol Device:R
- removed SW3, SW4: SW_Nidec_CAS-120A1, Button_Switch_SMD:Nidec_Copal_CAS-120A, symbol Switch:SW_Nidec_CAS-120A1
- added SW3, SW5: SW_SPDT, Button_Switch_SMD:SW_DPDT_CK_JS202011JCQN, symbol Switch:SW_SPDT
- C1, C2, C3, C4, C5, C6: footprint (none) -> Capacitor_SMD:C_0805_2012Metric_Pad1.18x1.45mm_HandSolder
- D1: footprint Diode_SMD:D_SOD-523 -> Diode_SMD:D_0805_2012Metric_Pad1.15x1.40mm_HandSolder
- J2: footprint (none) -> Connector_USB:USB_C_Receptacle_GCT_USB4105-xx-A_16P_TopMnt_Horizontal
- LD1, LD2, LD3, LD4, LD5, LD6, LD7: footprint LED_THT:LED_D5.0mm -> Connector_PinSocket_2.54mm:PinSocket_1x02_P2.54mm_Vertical
- LS1, R14, R16, R18, R20, R5, R7, R9: footprint (none) -> Connector_PinSocket_2.54mm:PinSocket_1x02_P2.54mm_Vertical
- Q1: footprint (none) -> Package_TO_SOT_SMD:TSOT-23_HandSoldering
- R1, R10, R12, R13, R15, R17, R19, R2, R21, R3, R4: footprint (none) -> Resistor_SMD:R_0805_2012Metric_Pad1.20x1.40mm_HandSolder
- R11: value R -> 91; footprint (none) -> Resistor_SMD:R_0805_2012Metric_Pad1.20x1.40mm_HandSolder
- R6: footprint (none) -> Resistor_THT:R_Axial_DIN0207_L6.3mm_D2.5mm_P15.24mm_Horizontal
- R8: footprint (none) -> Resistor_SMD:R_0805_2012Metric
- SW1, SW2: footprint (none) -> footprints 2:SWDIP2_256X170P100
- U1: footprint PCM_Espressif:ESP32-S2-SOLO -> ESP32_S2_SOLO_N4:XCVR_ESP32-S2-SOLO-N4
Connections:
- net +3.3V: now also SW3.1 (A), SW5.1 (A)
- net 3.3V_Switch: now also LD1.2 (A), LD2.2 (A), LD3.2 (A), LD4.2 (A), LD5.2 (A), LD6.2 (A), LD7.2 (A), SW3.2 (B); no longer R11.1
- net GND: now also R11.2, SW3.3 (C), SW5.3 (C); no longer LD1.1 (C), LD2.1 (C), LD3.1 (C), LD4.1 (C), LD5.1 (C), LD6.1 (C), LD7.1 (C)
- net at D1.1 (K), LS1.1: now also SW5.2 (B)
- new net Laser Ground: LD1.1 (C), LD2.1 (C), LD3.1 (C), LD4.1 (C), LD5.1 (C), LD6.1 (C), LD7.1 (C), R11.1

Commit message: Layout done
Changed lines of the file:
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@@
 		(color 0 0 0 0)
 	)
-	(junction
-		(at 49.53 99.06)
-		(diameter 0)
-		(color 0 0 0 0)
-	)
 	(no_connect
 		(at 220.98 114.3)
@@
 	(wire
 		(pts
+			(xy 39.37 218.44) (xy 39.37 219.71)
+		)
+		(stroke
+			(width 0)
+			(type default)
+		)
+	)
+	(wire
+		(pts
 			(xy 76.2 44.45) (xy 76.2 40.64)
 		)
@@
 	(wire
 		(pts
+			(xy 43.18 218.44) (xy 39.37 218.44)
+		)
+		(stroke
+			(width 0)
+			(type default)
+		)
+	)
+	(wire
+		(pts
 			(xy 49.53 99.06) (xy 58.42 99.06)
 		)
@@
 	(wire
 		(pts
+			(xy 45.72 147.32) (xy 41.91 147.32)
+		)
+		(stroke
+			(width 0)
+			(type default)
+		)
+	)
+	(wire
+		(pts
 			(xy 113.03 59.69) (xy 114.3 59.69)
 		)
@@
 	(wire
 		(pts
+			(xy 49.53 96.52) (xy 49.53 99.06)
+		)
+		(stroke
+			(width 0)
+			(type default)
+		)
+	)
+	(wire
+		(pts
 			(xy 226.06 224.79) (xy 226.06 228.6)
 		)
@@
 		(lib_name "GND_2")
 		(lib_id "power:GND")
-		(at 39.37 219.71 180)
+		(at 43.18 218.44 0)
 		(unit 1)
 		(exclude_from_sim no)
@@
 		(fields_autoplaced yes)
 		(property "Reference" "#PWR019"
-			(at 39.37 213.36 0)
+			(at 43.18 224.79 0)
 			(effects
 				(font
@@
 		)
 		(property "Value" "GND"
-			(at 39.37 214.63 0)
+			(at 43.18 223.52 0)
 			(effects
 				(font
@@
 		)
 		(property "Footprint" ""
-			(at 39.37 219.71 0)
+			(at 43.18 218.44 0)
 			(effects
 				(font
@@
 		)
 		(property "Datasheet" ""
-			(at 39.37 219.71 0)
+			(at 43.18 218.44 0)
 			(effects
 				(font
@@
 		)
 		(property "Description" "Power symbol creates a global label with name \"GND\" , ground"
-			(at 39.37 219.71 0)
+			(at 43.18 218.44 0)
 			(effects
 				(font
@@
 	(symbol
 		(lib_id "power:+5V")
-		(at 49.53 99.06 0)
+		(at 49.53 96.52 0)
 		(unit 1)
 		(exclude_from_sim no)
@@
 		(fields_autoplaced yes)
 		(property "Reference" "#PWR02"
-			(at 49.53 102.87 0)
+			(at 49.53 100.33 0)
 			(effects
 				(font
@@
 		)
 		(property "Value" "+5V"
-			(at 49.53 95.25 0)
+			(at 49.53 92.71 0)
 			(effects
 				(font
@@
 		)
 		(property "Footprint" ""
-			(at 49.53 99.06 0)
+			(at 49.53 96.52 0)
 			(effects
 				(font
@@
 		)
 		(property "Datasheet" ""
-			(at 49.53 99.06 0)
+			(at 49.53 96.52 0)
 			(effects
 				(font
@@
 		)
 		(property "Description" ""
-			(at 49.53 99.06 0)
+			(at 49.53 96.52 0)
 			(effects
 				(font
@@
 		(lib_name "GND_3")
 		(lib_id "power:GND")
-		(at 41.91 147.32 180)
+		(at 45.72 147.32 0)
 		(unit 1)
 		(exclude_from_sim no)
@@
 		(fields_autoplaced yes)
 		(property "Reference" "#PWR018"
-			(at 41.91 140.97 0)
+			(at 45.72 153.67 0)
 			(effects
 				(font
@@
 		)
 		(property "Value" "GND"
-			(at 41.91 142.24 0)
+			(at 45.72 152.4 0)
 			(effects
 				(font
@@
 		)
 		(property "Footprint" ""
-			(at 41.91 147.32 0)
+			(at 45.72 147.32 0)
 			(effects
 				(font
@@
 		)
 		(property "Datasheet" ""
-			(at 41.91 147.32 0)
+			(at 45.72 147.32 0)
 			(effects
 				(font
@@
 		)
 		(property "Description" "Power symbol creates a global label with name \"GND\" , ground"
-			(at 41.91 147.32 0)
+			(at 45.72 147.32 0)
 			(effects
 				(font

Commit message: I2S speaker and ESD protection schematic and footprints added
Parts:
- added C10: 0.1uF, Capacitor_SMD:C_0805_2012Metric_Pad1.18x1.45mm_HandSolder, symbol Device:C
- added C7, C8: 220pF, Capacitor_SMD:C_0805_2012Metric_Pad1.18x1.45mm_HandSolder, symbol Device:C
- added C9: 10uF, Capacitor_SMD:C_0805_2012Metric_Pad1.18x1.45mm_HandSolder, symbol Device:C
- added D2, D3: SMAJ5.0CA, Diode_SMD:D_0805_2012Metric_Pad1.15x1.40mm_HandSolder, symbol Diode:SMAJ5.0CA
- added D4: D, Diode_SMD:D_0805_2012Metric_Pad1.15x1.40mm_HandSolder, symbol Device:D
- added D5: D_Schottky, Diode_SMD:D_0805_2012Metric_Pad1.15x1.40mm_HandSolder, symbol Device:D_Schottky
- added F1: Polyfuse, Diode_SMD:D_0805_2012Metric_Pad1.15x1.40mm_HandSolder, symbol Device:Polyfuse
- added LS2: Speaker, Connector_PinSocket_2.54mm:PinSocket_1x02_P2.54mm_Vertical, symbol Device:Speaker
- added R22: 1M, Resistor_SMD:R_0805_2012Metric_Pad1.20x1.40mm_HandSolder, symbol Device:R
- added U4: MAX98357A, Package_DFN_QFN:TQFN-16-1EP_3x3mm_P0.5mm_EP1.23x1.23mm, symbol Audio:MAX98357A
Connections:
- net +3.3V: now also C10.1, C9.1, R22.1, U4.7 (VDD), U4.8 (VDD)
- net +5V: now also F1.1; no longer C1.1, U2.3 (VI)
- net D+: now also D2.2 (A2)
- net D-: now also D3.2 (A2)
- net GND: now also C10.2, C7.2, C8.2, C9.2, D2.1 (A1), D3.1 (A1), D5.2 (A), U4.11 (GND), U4.15 (GND), U4.17 (PAD), U4.3 (GND)
- net I2S1: now reaches U1.17 (GPIO9/TOUCH9/ADC1_CH8/FSPIHD)
- net I2S1: now also U4.1 (DIN)
- net I2S2: now reaches U1.18 (GPIO10/TOUCH10/ADC1_CH9/FSPICS0/FSPIIO4)
- net I2S2: now also U4.16 (BCLK)
- net I2S3: now reaches U1.19 (GPIO11/TOUCH11/ADC2_CH0/FSPID/FSPIIO5)
- net I2S3: now also U4.14 (LRCLK)
- new net: C7.1, LS2.1, U4.10 (OUTN)
- new net: D4.2 (A), F1.2
- new net: C8.1, LS2.2, U4.9 (OUTP)
- new net: R22.2, U4.4 (~{SD_MODE})
- new net ESD Protected 5V: C1.1, D4.1 (K), D5.1 (K), U2.3 (VI)
- no-connect marks 30 -> 28
Other:
- moved on the sheet: D1, LS1, Q1, R12, R13, R6, SW3, SW5

Commit message: Final project submission
Parts:
- added TP1, TP2, TP3: TestPoint, TestPoint:TestPoint_Plated_Hole_D2.0mm, symbol Connector:TestPoint
- D2, D3: footprint Diode_SMD:D_0805_2012Metric_Pad1.15x1.40mm_HandSolder -> Diode_SMD:D_SOD-323_HandSoldering
Connections:
- net +3.3V: now also TP2.1
- net +5V: now also TP1.1
- net ESD Protected 5V: now also TP3.1
Other:
- note added: "7 Photoresistors for light sensing"
- note added: "7 lasers to be the strings of our laser harp"
- note added: "Comparators to filter out noise and in case the ADC pins do not work as expected"
- note added: "ESD Protection"
- note added: "Speaker driven by MAX98357 chip using I2S"
- note added: "Speaker driven directly by GPIO"
- note added: "Switch to control lasers"
- note added: "Voltage divider for reference voltage at 3/4 VDD"
